File: Pumpkin-Monitor.kicad_pcb (KiCad board)
At the start: 2 copper layers, 46.4 x 50.6 mm, 73 parts, among them J1 USB_A, Q1 SS8050, Q2 SS8050, Q3 SS8050, SW1 KMR221GLFS, SW2 KMR221GLFS, U1 XC6206P182MR, U2 AMS1117-3.3, U3 CH343P, U4 W25Q32JVSS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

Commit message: corrected GND connection of ESP8266 ( added vias to bulky polygons )
Routing:
- net Earth: vias 111 -> 115
Changed lines of the file:
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@@
 				(font
 					(size 0.001 0.001)
+					(thickness 0.15)
 				)
 			)
@@
 				(font
 					(size 0.001 0.001)
+					(thickness 0.15)
 				)
 			)
@@
 	)
 	(via
+		(at 177.65 125.4)
+		(size 0.45)
+		(drill 0.3)
+		(layers "F.Cu" "B.Cu")
+		(free yes)
+		(net 1)
+	)
+	(via
 		(at 192.7 102.2)
 		(size 0.45)
@@
 	)
 	(via
+		(at 177 125.65)
+		(size 0.45)
+		(drill 0.3)
+		(layers "F.Cu" "B.Cu")
+		(free yes)
+		(net 1)
+	)
+	(via
 		(at 180.85 127.85)
 		(size 0.45)
@@
 	)
 	(via
+		(at 176.2 125.85)
+		(size 0.45)
+		(drill 0.3)
+		(layers "F.Cu" "B.Cu")
+		(free yes)
+		(net 1)
+	)
+	(via
 		(at 184.15 120.45)
 		(size 0.45)
@@
 		(net 1)
 	)
+	(via
+		(at 177.4 124.25)
+		(size 0.45)
+		(drill 0.3)
+		(layers "F.Cu" "B.Cu")
+		(free yes)
+		(net 1)
+	)
